File: adapters/raspberry-pi/raspberry-pi-adapter.kicad_pcb (KiCad board)
At the start: 2 copper layers, 65 x 56 mm, 17 parts, among them J2 Bus_M.2_Socket_E, J3 Raspberry_Pi_4, U1 SN74AXC4T245PW, U2 TLV70018_SOT23-5

Commit message: Fixed a few Errors in the PCBs and added Notice that Audio sounds weird
Parts:
- moved R1 10.8 mm to (114.8, 78.4)
- moved R2 4.53 mm to (126.0, 79.1)
Connections:
- J2 pad 58: /SCL -> /SDA
- J2 pad 60: /SDA -> /SCL
- U1 pad 6: /PCM_DOUT_1V8 -> /PCM_DIN_1V8
Routing:
- net /PCM_DOUT_1V8: track 8.83 -> 0.00 mm
- net /PCM_DIN_1V8: track 0.00 -> 8.63 mm
- net +3V3: track 93.8 -> 98.8 mm, vias 4 -> 3
- net /SCL: track 23.8 -> 20.7 mm
- net GND: vias 3 -> 75
