File: adapters/raspberry-pi/raspberry-pi-adapter.kicad_sch (KiCad schematic)
At the start: 18 parts, among them J2 Bus_M.2_Socket_E, J3 Raspberry_Pi_4, M1 M.2 Solder Nut, U1 SN74AXC4T245PW, U2 TLV70018_SOT23-5

Commit message: Fixed a few Errors in the PCBs and added Notice that Audio sounds weird
Connections:
- net SCL: now also J2.60 (I2C_CLK); no longer J2.58 (I2C_DATA)
- net SDA: now also J2.58 (I2C_DATA); no longer J2.60 (I2C_CLK)
