File: pcb/Si4689.kicad_sch (KiCad schematic)
At the start: 35 parts, among them J2 ANT0, U4 Si4689-A10, U5 ZD25WQ32C, Y1 19.2MHZ

Commit message: Fixed a few Errors in the PCBs and added Notice that Audio sounds weird
Parts:
- removed TP3: LOOP_N, TestPoint:TestPoint_Pad_D1.0mm, symbol Connector:TestPoint
- removed TP4: LOOP_P, TestPoint:TestPoint_Pad_D1.0mm, symbol Connector:TestPoint
Connections:
- no-connect marks 2 -> 4
