File: pcb/Si468x.kicad_pcb (KiCad board)
At the start: 4 copper layers, 22 x 30 mm, 60 parts, among them J1 Bus_M.2_Socket_E, J2 ANT0, Q1 BSS138, U1 TPS7A2118-DRB, U2 PCA9306, U3 74LVC1G17, U4 Si4689-A10, U5 ZD25WQ32C, Y1 19.2MHZ

Commit message: Fixed a few Errors in the PCBs and added Notice that Audio sounds weird
Parts:
- removed R1, R2, R3: 33R, Resistor_SMD:R_0402_1005Metric
- removed TP3: LOOP_N, TestPoint:TestPoint_Pad_D1.0mm
- removed TP4: LOOP_P, TestPoint:TestPoint_Pad_D1.0mm
- moved R7 3.31 mm to (153.2, 97.3)
- moved C13 1.02 mm to (148.6, 86.2)
Connections:
- J1 pad 10: Net-(J1-PCM_SYNC/I2S_WS) -> /Si4689/DFS
- J1 pad 12: Net-(J1-PCM_IN/I2S_SD_IN) -> /Si4689/DOUT
- J1 pad 8: Net-(J1-PCM_CLK/I2S_SCK) -> /Si4689/DCLK
- Q1 pad 1: /Si4689/INTB -> +1V8
- U4 pad 6: Net-(U4-LOOP_N) -> unconnected-(U4-LOOP_N-Pad6)
- U4 pad 7: Net-(U4-LOOP_P) -> unconnected-(U4-LOOP_P-Pad7)
Routing:
- net Net-(U4-LOOP_N): track 6.30 -> 0.00 mm
- net Net-(U4-LOOP_P): track 5.00 -> 0.00 mm
- net /Si4689/DOUT: track 16.6 -> 21.1 mm
- net /Si4689/DFS: track 19.7 -> 24.1 mm
- net /Si4689/DCLK: track 20.8 -> 25.0 mm
- net Net-(J1-PCM_IN/I2S_SD_IN): track 3.54 -> 0.00 mm
- net Net-(J1-PCM_SYNC/I2S_WS): track 3.34 -> 0.00 mm
- net Net-(J1-PCM_CLK/I2S_SCK): track 3.13 -> 0.00 mm
- net /Si4689/INTB: track 12.4 -> 9.79 mm
- net Net-(U4-XTALO): track 9.74 -> 7.83 mm, vias 2 -> 0
- net Net-(U4-DACREF): track 2.24 -> 1.37 mm
