File: pcb/Si468x.kicad_sch (KiCad schematic)
At the start: 25 parts, among them J1 Bus_M.2_Socket_E, Q1 BSS138, U1 TPS7A2118-DRB, U2 PCA9306, U3 74LVC1G17

Commit message: Fixed a few Errors in the PCBs and added Notice that Audio sounds weird
Parts:
- removed R1, R2, R3: 33R, Resistor_SMD:R_0402_1005Metric, symbol Device:R
Connections:
- net +1V8: now also Q1.1 (G)
- net Si4689/DCLK: now also J1.8 (PCM_CLK/I2S_SCK)
- net Si4689/DFS: now also J1.10 (PCM_SYNC/I2S_WS)
- net Si4689/DOUT: now also J1.12 (PCM_IN/I2S_SD_IN)
- net Si4689/INTB: no longer Q1.1 (G)
